File: Production/SparkFun_Lil_Soundie_Audio_Player-Panel_v10.brd (EAGLE design)
At the start: 302.8 x 142.7 mm, 1606 parts, among them J1 Audio Jack, J10 AMP FCI 10103594-0001LF, J13 Audio Jack, J14 AMP FCI 10103594-0001LF, J17 Audio Jack, J18 AMP FCI 10103594-0001LF, J2 AMP FCI 10103594-0001LF, J21 Audio Jack, J22 AMP FCI 10103594-0001LF, J25 Audio Jack, J26 AMP FCI 10103594-0001LF, J29 Audio Jack, J30 AMP FCI 10103594-0001LF, J33 Audio Jack, J34 AMP FCI 10103594-0001LF, J37 Audio Jack, J38 AMP FCI 10103594-0001LF, J41 Audio Jack, J42 AMP FCI 10103594-0001LF, J45 Audio Jack, J46 AMP FCI 10103594-0001LF, J49 Audio Jack, J5 Audio Jack, J50 AMP FCI 10103594-0001LF, J53 Audio Jack, J54 AMP FCI 10103594-0001LF, J57 Audio Jack, J58 AMP FCI 10103594-0001LF, J6 AMP FCI 10103594-0001LF, J61 Audio Jack, J62 AMP FCI 10103594-0001LF, J65 Audio Jack, J66 AMP FCI 10103594-0001LF, J69 Audio Jack, J70 AMP FCI 10103594-0001LF, J73 Audio Jack, J74 AMP FCI 10103594-0001LF, J77 Audio Jack, J78 AMP FCI 10103594-0001LF, J81 Audio Jack, J82 AMP FCI 10103594-0001LF, J85 Audio Jack, J86 AMP FCI 10103594-0001LF, J89 Audio Jack, J9 Audio Jack, J90 AMP FCI 10103594-0001LF, J93 Audio Jack, J94 AMP FCI 10103594-0001LF, J97 Audio Jack, J98 AMP FCI 10103594-0001LF, U1 VS1000D, U10 4MB Flash, U11 VS1000D, U12 4MB Flash, U13 VS1000D, U14 4MB Flash, U15 VS1000D, U16 4MB Flash, U17 VS1000D, U18 4MB Flash, U19 VS1000D, U2 VS1000D, U20 4MB Flash, U21 VS1000D, U22 4MB Flash, U23 VS1000D, U24 4MB Flash, U25 VS1000D, U26 4MB Flash, U27 VS1000D, U28 4MB Flash, U29 VS1000D, U3 4MB Flash, U30 4MB Flash, U31 VS1000D, U32 4MB Flash, U33 VS1000D, U34 4MB Flash, U35 VS1000D, U36 4MB Flash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

Commit message: created panel v10
Parts:
- removed C361, C362, C379, C380, C397, C398, C415, C416, C433, C434: 22pF, SparkFun-Capacitors:0603-CAP
- removed C363, C366, C367, C368, C369, C370, C371, C381, C384, C385, C386, C387, C388, C389, C399, C402, C403, C404, C405, C406, C407, C417, C420, C421, C422, C423, C424, C425, C435, C438, C439, C440, C441, C442, C443: 0.1uF, SparkFun-Capacitors:0603-CAP
- removed C364, C372, C382, C390, C400, C408, C418, C426, C436, C444: 1.0uF, SparkFun-Capacitors:0603-CAP
- removed C365, C373, C374, C375, C383, C391, C392, C393, C401, C409, C410, C411, C419, C427, C428, C429, C437, C445, C446, C447: 10uF, SparkFun-Capacitors:0603-CAP
- removed C376, C377, C394, C395, C412, C413, C430, C431, C448, C449: 10nF, SparkFun-Capacitors:0603-CAP
- removed C378, C396, C414, C432, C450: 47nF, SparkFun-Capacitors:0603-CAP
- removed D100, D84, D88, D92, D96: PESD1CAN, SparkFun-DiscreteSemi:SOT23-3
- removed D81, D82, D85, D86, D89, D90, D93, D94, D97, D98: 1A/23V/620mV, SparkFun-DiscreteSemi:SOD-323
- removed D83, D87, D91, D95, D99: RED, SparkFun-LED:LED-0603
- removed E$5, E$8: (no value), SparkFun-Aesthetics:FIDUCIAL-1X2
- removed FD100, FD81, FD82, FD83, FD84, FD85, FD86, FD87, FD88, FD89, FD90, FD91, FD92, FD93, FD94, FD95, FD96, FD97, FD98, FD99: FIDUCIALUFIDUCIAL, SparkFun-Aesthetics:FIDUCIAL-MICRO
- removed H41, H42, H43, H44, H45, H46, H47, H48, H49, H50: STAND-OFFTIGHT, SparkFun-Electromechanical:STAND-OFF-TIGHT
- removed J100, J84, J88, J92, J96: (no value), SparkFun-Connectors:1X06
- removed J81, J85, J89, J93, J97: Audio Jack, SparkFun-Connectors:AUDIO-JACK-3.5MM-SMD
- removed J82, J86, J90, J94, J98: AMP FCI 10103594-0001LF, SparkFun-Connectors:USB-MICROB-PTH
- removed J83, J87, J91, J95, J99: (no value), SparkFun-Connectors:1X08
- removed LOGO41, LOGO43, LOGO45, LOGO47, LOGO49: OSHW-LOGOL, SparkFun-Aesthetics:OSHW-LOGO-L
- removed LOGO42, LOGO44, LOGO46, LOGO48, LOGO50: SFE_LOGO_NAME.1_INCH, SparkFun-Aesthetics:SFE_LOGO_NAME_.1
- removed R501, R502, R503, R505, R526, R527, R528, R530, R551, R552, R553, R555, R576, R577, R578, R580, R601, R602, R603, R605: 1M, SparkFun-Resistors:0603-RES
- removed R504, R506, R515, R523, R524, R525, R529, R531, R540, R548, R549, R550, R554, R556, R565, R573, R574, R575, R579, R581, R590, R598, R599, R600, R604, R606, R615, R623, R624, R625: 100k, SparkFun-Resistors:0603-RES
- removed R507, R532, R557, R582, R607: 150K, SparkFun-Resistors:0603-RES
- removed R508, R509, R533, R534, R558, R559, R583, R584, R608, R609: 10K, SparkFun-Resistors:0603-RES
- removed R510, R511, R535, R536, R560, R561, R585, R586, R610, R611: 470, SparkFun-Resistors:0603-RES
- removed R512, R513, R537, R538, R562, R563, R587, R588, R612, R613: 20, SparkFun-Resistors:0603-RES
- removed R514, R539, R564, R589, R614: 180, SparkFun-Resistors:0603-RES
- removed R516, R517, R518, R519, R520, R521, R541, R542, R543, R544, R545, R546, R566, R567, R568, R569, R570, R571, R591, R592, R593, R594, R595, R596, R616, R617, R618, R619, R620, R621: 100k, SparkFun-Resistors:0603
- removed R522, R547, R572, R597, R622: 10, SparkFun-Resistors:0603-RES
- removed S21, S22, S23, S24, S25: SWITCH-MOMENTARY-2SMD, SparkFun-Electromechanical:TACTILE-SWITCH-SMD
- removed U$21, U$22, U$23, U$24, U$25: (no value), SparkFun-Aesthetics:SFE_LOGO_FLAME_.1
- removed U41, U43, U45, U47, U49: VS1000D, SparkFun-IC-Conversion:LQFP-48
- removed U42, U44, U46, U48, U50: 4MB Flash, SparkFun-IC-Memory:SO08
- removed Y21, Y22, Y23, Y24, Y25: 12MHz, SparkFun-FreqCtrl:CRYSTAL-SMD-5X3
- added E$6, E$7: (no value), SparkFun-Aesthetics:FIDUCIAL-1X2
- E$1, E$2: device SparkFun-Retired:FIDUCIAL-1.5X3 -> SparkFun-Aesthetics:FIDUCIAL-1X2
- E$3, E$4: device SparkFun-Aesthetics:FIDUCIAL-1X2 -> SparkFun-Retired:FIDUCIAL-1.5X3
- moved H31 304.8 mm to (2.54, 226.3), turned to 270 degrees
- moved H32 303.7 mm to (22.9, 226.3), turned to 270 degrees
- moved D63 302.6 mm to (17.9, 225.5), turned to 0 degrees
- moved FD62 300.5 mm to (1.08, 223.1), turned to 270 degrees
- moved S16 300.0 mm to (12.7, 223.5), turned to 0 degrees
- moved R382 299.8 mm to (8.06, 223.2), turned to 90 degrees
- moved D61 299.5 mm to (6.35, 222.8), turned to 270 degrees
- moved FD64 298.3 mm to (1.11, 221.6), turned to 0 degrees
- moved R389 298.0 mm to (17.5, 222.3), turned to 90 degrees
- moved C276 294.9 mm to (8.15, 219.7), turned to 180 degrees
- moved C275 294.8 mm to (11.3, 219.8), turned to 0 degrees
- moved C279 294.6 mm to (14.4, 219.8), turned to 180 degrees
- moved C282 294.3 mm to (18.1, 219.7), turned to 0 degrees
- moved C283 293.3 mm to (5.71, 218.4), turned to 270 degrees
- moved C274 293.0 mm to (8.10, 218.4), turned to 0 degrees
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Connections:
- removed net AVDD20: C365.1, C366.1, C367.1, C368.1, R502.2, R503.2, U41.34, U41.39, U41.44, U41.46
- removed net AVDD21: C383.1, C384.1, C385.1, C386.1, R527.2, R528.2, U43.34, U43.39, U43.44, U43.46
- removed net AVDD22: C401.1, C402.1, C403.1, C404.1, R552.2, R553.2, U45.34, U45.39, U45.44, U45.46
- removed net AVDD23: C419.1, C420.1, C421.1, C422.1, R577.2, R578.2, U47.34, U47.39, U47.44, U47.46
- removed net AVDD24: C437.1, C438.1, C439.1, C440.1, R602.2, R603.2, U49.34, U49.39, U49.44, U49.46
- removed net CVDD20: C369.1, C372.1, R505.2, U41.32
- removed net CVDD21: C387.1, C390.1, R530.2, U43.32
- removed net CVDD22: C405.1, C408.1, R555.2, U45.32
- removed net CVDD23: C423.1, C426.1, R580.2, U47.32
- removed net CVDD24: C441.1, C444.1, R605.2, U49.32
- removed net DVDD20: C363.1, C370.1, C371.1, R504.2, R506.2, R515.2, R523.1, R524.2, U41.19, U41.30, U41.7, U42.3, U42.7, U42.8
- removed net DVDD21: C381.1, C388.1, C389.1, R529.2, R531.2, R540.2, R548.1, R549.2, U43.19, U43.30, U43.7, U44.3, U44.7, U44.8
- removed net DVDD22: C399.1, C406.1, C407.1, R554.2, R556.2, R565.2, R573.1, R574.2, U45.19, U45.30, U45.7, U46.3, U46.7, U46.8
- removed net DVDD23: C417.1, C424.1, C425.1, R579.2, R581.2, R590.2, R598.1, R599.2, U47.19, U47.30, U47.7, U48.3, U48.7, U48.8
- removed net DVDD24: C435.1, C442.1, C443.1, R604.2, R606.2, R615.2, R623.1, R624.2, U49.19, U49.30, U49.7, U50.3, U50.7, U50.8
- removed net GBUF20: R522.1, U41.43
- removed net GBUF21: R547.1, U43.43
- removed net GBUF22: R572.1, U45.43
- removed net GBUF23: R597.1, U47.43
- removed net GBUF24: R622.1, U49.43
- removed net GND20: C361.1, C362.1, C363.2, C364.2, C365.2, C366.2, C367.2, C368.2, C369.2, C370.2, C371.2, C372.2, C373.1, C376.2, C377.2, C378.2, D83.C, D84.3, J81.SLEEVE, J82.GND, J83.2, J84.4, R505.1, R507.1, R508.1, R509.1, R516.2, R517.2, R518.2, R519.2, R520.2, R521.2, R525.2, U41.18, U41.31, U41.38, U41.41, U41.42, U41.48, U41.6, U41.8, U42.4
- removed net GND21: C379.1, C380.1, C381.2, C382.2, C383.2, C384.2, C385.2, C386.2, C387.2, C388.2, C389.2, C390.2, C391.1, C394.2, C395.2, C396.2, D87.C, D88.3, J85.SLEEVE, J86.GND, J87.2, J88.4, R530.1, R532.1, R533.1, R534.1, R541.2, R542.2, R543.2, R544.2, R545.2, R546.2, R550.2, U43.18, U43.31, U43.38, U43.41, U43.42, U43.48, U43.6, U43.8, U44.4
- removed net GND22: C397.1, C398.1, C399.2, C400.2, C401.2, C402.2, C403.2, C404.2, C405.2, C406.2, C407.2, C408.2, C409.1, C412.2, C413.2, C414.2, D91.C, D92.3, J89.SLEEVE, J90.GND, J91.2, J92.4, R555.1, R557.1, R558.1, R559.1, R566.2, R567.2, R568.2, R569.2, R570.2, R571.2, R575.2, U45.18, U45.31, U45.38, U45.41, U45.42, U45.48, U45.6, U45.8, U46.4
- removed net GND23: C415.1, C416.1, C417.2, C418.2, C419.2, C420.2, C421.2, C422.2, C423.2, C424.2, C425.2, C426.2, C427.1, C430.2, C431.2, C432.2, D95.C, D96.3, J93.SLEEVE, J94.GND, J95.2, J96.4, R580.1, R582.1, R583.1, R584.1, R591.2, R592.2, R593.2, R594.2, R595.2, R596.2, R600.2, U47.18, U47.31, U47.38, U47.41, U47.42, U47.48, U47.6, U47.8, U48.4
- removed net GND24: C433.1, C434.1, C435.2, C436.2, C437.2, C438.2, C439.2, C440.2, C441.2, C442.2, C443.2, C444.2, C445.1, C448.2, C449.2, C450.2, D100.3, D99.C, J100.4, J97.SLEEVE, J98.GND, J99.2, R605.1, R607.1, R608.1, R609.1, R616.2, R617.2, R618.2, R619.2, R620.2, R621.2, R625.2, U49.18, U49.31, U49.38, U49.41, U49.42, U49.48, U49.6, U49.8, U50.4
- removed net IO_160: J83.8, R521.1, U41.10
- removed net IO_161: J83.3, R516.1, U41.2
- removed net IO_162: J83.4, R517.1, U41.3
- removed net IO_163: J83.6, R519.1, U41.5
- removed net IO_164: J83.7, R520.1, U41.9
- removed net IO_165: R525.1, U41.11
- removed net IO_166: J83.5, R518.1, U41.4
- removed net IO_167: R515.1, U41.12
- removed net IO_168: J87.8, R546.1, U43.10
- removed net IO_169: J87.3, R541.1, U43.2
- removed net IO_170: J87.4, R542.1, U43.3
- removed net IO_171: J87.6, R544.1, U43.5
- removed net IO_172: J87.7, R545.1, U43.9
- removed net IO_173: R550.1, U43.11
- removed net IO_174: J87.5, R543.1, U43.4
- removed net IO_175: R540.1, U43.12
- removed net IO_176: J91.8, R571.1, U45.10
- removed net IO_177: J91.3, R566.1, U45.2
- removed net IO_178: J91.4, R567.1, U45.3
- removed net IO_179: J91.6, R569.1, U45.5
- removed net IO_180: J91.7, R570.1, U45.9
- removed net IO_181: R575.1, U45.11
- removed net IO_182: J91.5, R568.1, U45.4
- removed net IO_183: R565.1, U45.12
- removed net IO_184: J95.8, R596.1, U47.10
- removed net IO_185: J95.3, R591.1, U47.2
- removed net IO_186: J95.4, R592.1, U47.3
- removed net IO_187: J95.6, R594.1, U47.5
- removed net IO_188: J95.7, R595.1, U47.9
- removed net IO_189: R600.1, U47.11
- removed net IO_190: J95.5, R593.1, U47.4
- removed net IO_191: R590.1, U47.12
- removed net IO_192: J99.8, R621.1, U49.10
- removed net IO_193: J99.3, R616.1, U49.2
- removed net IO_194: J99.4, R617.1, U49.3
- removed net IO_195: J99.6, R619.1, U49.5
- removed net IO_196: J99.7, R620.1, U49.9
- removed net IO_197: R625.1, U49.11
- removed net IO_198: J99.5, R618.1, U49.4
- removed net IO_199: R615.1, U49.12
- removed net LEFT20: R510.2, R513.2, U41.47
- removed net LEFT21: R535.2, R538.2, U43.47
- removed net LEFT22: R560.2, R563.2, U45.47
- removed net LEFT23: R585.2, R588.2, U47.47
- removed net LEFT24: R610.2, R613.2, U49.47
- removed net L_AC20: C374.2, J81.TIP, J84.5, R509.2
- removed net L_AC21: C392.2, J85.TIP, J88.5, R534.2
- removed net L_AC22: C410.2, J89.TIP, J92.5, R559.2
- removed net L_AC23: C428.2, J93.TIP, J96.5, R584.2
- removed net L_AC24: C446.2, J100.5, J97.TIP, R609.2
- removed net N$224: C364.1, U41.45
- removed net N$225: C373.2, R506.1, U41.1
- removed net N$226: D82.A, J82.VBUS
- removed net N$227: D83.A, R514.2
- removed net N$228: C374.1, R510.1
- removed net N$229: C376.1, R513.1
- removed net N$230: C375.1, R511.1
- removed net N$231: C377.1, R512.1
- removed net N$232: C378.1, R522.2
- removed net N$233: R504.1
- removed net N$234: C382.1, U43.45
- removed net N$235: C391.2, R531.1, U43.1
- removed net N$236: D86.A, J86.VBUS
- removed net N$237: D87.A, R539.2
- removed net N$238: C392.1, R535.1
- removed net N$239: C394.1, R538.1
- removed net N$240: C393.1, R536.1
- removed net N$241: C395.1, R537.1
- removed net N$242: C396.1, R547.2
- removed net N$243: R529.1
- removed net N$244: C400.1, U45.45
- removed net N$245: C409.2, R556.1, U45.1
- removed net N$246: D90.A, J90.VBUS
- removed net N$247: D91.A, R564.2
- removed net N$248: C410.1, R560.1
- removed net N$249: C412.1, R563.1
- removed net N$250: C411.1, R561.1
- removed net N$251: C413.1, R562.1
- removed net N$252: C414.1, R572.2
- removed net N$253: R554.1
- removed net N$254: C418.1, U47.45
- removed net N$255: C427.2, R581.1, U47.1
- removed net N$256: D94.A, J94.VBUS
- removed net N$257: D95.A, R589.2
- removed net N$258: C428.1, R585.1
- removed net N$259: C430.1, R588.1
- removed net N$260: C429.1, R586.1
- removed net N$261: C431.1, R587.1
- removed net N$262: C432.1, R597.2
- removed net N$263: R579.1
- removed net N$264: C436.1, U49.45
- removed net N$265: C445.2, R606.1, U49.1
- removed net N$266: D98.A, J98.VBUS
- removed net N$267: D99.A, R614.2
- removed net N$268: C446.1, R610.1
- removed net N$269: C448.1, R613.1
- removed net N$270: C447.1, R611.1
- removed net N$271: C449.1, R612.1
- removed net N$272: C450.1, R622.2
- removed net N$273: R604.1
- removed net PWRBTN20: J84.1, R507.2, S21.3, U41.37
- removed net PWRBTN21: J88.1, R532.2, S22.3, U43.37
- removed net PWRBTN22: J92.1, R557.2, S23.3, U45.37
- removed net PWRBTN23: J96.1, R582.2, S24.3, U47.37
- removed net PWRBTN24: J100.1, R607.2, S25.3, U49.37
- removed net RDY20: R523.2, U41.13
- removed net RDY21: R548.2, U43.13
- removed net RDY22: R573.2, U45.13
- removed net RDY23: R598.2, U47.13
- removed net RDY24: R623.2, U49.13
- removed net RIGHT20: R511.2, R512.2, U41.40
- removed net RIGHT21: R536.2, R537.2, U43.40
- removed net RIGHT22: R561.2, R562.2, U45.40
- removed net RIGHT23: R586.2, R587.2, U47.40
- removed net RIGHT24: R611.2, R612.2, U49.40
- removed net RX20: J84.2, U41.27
- removed net RX21: J88.2, U43.27
- removed net RX22: J92.2, U45.27
- removed net RX23: J96.2, U47.27
- removed net RX24: J100.2, U49.27
- removed net R_AC20: C375.2, J81.RING, J84.6, R508.2
- removed net R_AC21: C393.2, J85.RING, J88.6, R533.2
- removed net R_AC22: C411.2, J89.RING, J92.6, R558.2
- removed net R_AC23: C429.2, J93.RING, J96.6, R583.2
- removed net R_AC24: C447.2, J100.6, J97.RING, R608.2
- removed net SCLK20: U41.23, U42.6
- removed net SCLK21: U43.23, U44.6
- removed net SCLK22: U45.23, U46.6
- removed net SCLK23: U47.23, U48.6
- removed net SCLK24: U49.23, U50.6
- removed net SI20: U41.24, U42.2
- removed net SI21: U43.24, U44.2
- removed net SI22: U45.24, U46.2
- removed net SI23: U47.24, U48.2
- removed net SI24: U49.24, U50.2
- removed net SO20: U41.25, U42.5
- removed net SO21: U43.25, U44.5
- removed net SO22: U45.25, U46.5
- removed net SO23: U47.25, U48.5
- removed net SO24: U49.25, U50.5
- removed net TX20: J84.3, U41.26
- removed net TX21: J88.3, U43.26
- removed net TX22: J92.3, U45.26
- removed net TX23: J96.3, U47.26
- removed net TX24: J100.3, U49.26
- removed net USBN20: D84.1, J82.D-, R502.1, U41.36
- removed net USBN21: D88.1, J86.D-, R527.1, U43.36
- removed net USBN22: D92.1, J90.D-, R552.1, U45.36
- removed net USBN23: D96.1, J94.D-, R577.1, U47.36
- removed net USBN24: D100.1, J98.D-, R602.1, U49.36
- removed net USBP20: D84.2, J82.D+, R503.1, U41.35
- removed net USBP21: D88.2, J86.D+, R528.1, U43.35
- removed net USBP22: D92.2, J90.D+, R553.1, U45.35
- removed net USBP23: D96.2, J94.D+, R578.1, U47.35
- removed net USBP24: D100.2, J98.D+, R603.1, U49.35
- removed net VCC20: D81.A, J83.1
- removed net VCC21: D85.A, J87.1
- removed net VCC22: D89.A, J91.1
- removed net VCC23: D93.A, J95.1
- removed net VCC24: D97.A, J99.1
- removed net VHIGH20: D81.C, D82.C, R514.1, S21.1, U41.33
- removed net VHIGH21: D85.C, D86.C, R539.1, S22.1, U43.33
- removed net VHIGH22: D89.C, D90.C, R564.1, S23.1, U45.33
- removed net VHIGH23: D93.C, D94.C, R589.1, S24.1, U47.33
- removed net VHIGH24: D97.C, D98.C, R614.1, S25.1, U49.33
- removed net XCS20: R524.1, U41.22, U42.1
- removed net XCS21: R549.1, U43.22, U44.1
- removed net XCS22: R574.1, U45.22, U46.1
- removed net XCS23: R599.1, U47.22, U48.1
- removed net XCS24: R624.1, U49.22, U50.1
- removed net XTAL40: C361.2, R501.2, U41.28, Y21.3
- removed net XTAL41: C362.2, R501.1, U41.29, Y21.1
- removed net XTAL42: C379.2, R526.2, U43.28, Y22.3
- removed net XTAL43: C380.2, R526.1, U43.29, Y22.1
- removed net XTAL44: C397.2, R551.2, U45.28, Y23.3
- removed net XTAL45: C398.2, R551.1, U45.29, Y23.1
- removed net XTAL46: C415.2, R576.2, U47.28, Y24.3
- removed net XTAL47: C416.2, R576.1, U47.29, Y24.1
- removed net XTAL48: C433.2, R601.2, U49.28, Y25.3
- removed net XTAL49: C434.2, R601.1, U49.29, Y25.1
Routing:
- net GND21: track 103.7 -> 0.00 mm, vias 45 -> 0
- net GND24: track 103.7 -> 0.00 mm, vias 45 -> 0
- net GND22: track 103.7 -> 0.00 mm, vias 45 -> 0
- net GND20: track 103.7 -> 0.00 mm, vias 45 -> 0
- net GND23: track 103.7 -> 0.00 mm, vias 45 -> 0
- net DVDD23: track 81.4 -> 0.00 mm, vias 5 -> 0
- net DVDD21: track 81.4 -> 0.00 mm, vias 5 -> 0
- net DVDD20: track 81.4 -> 0.00 mm, vias 5 -> 0
- net DVDD24: track 81.4 -> 0.00 mm, vias 5 -> 0
- net DVDD22: track 81.4 -> 0.00 mm, vias 5 -> 0
- net VHIGH24: track 67.9 -> 0.00 mm, vias 2 -> 0
- net VHIGH23: track 67.9 -> 0.00 mm, vias 2 -> 0
- net VHIGH21: track 67.9 -> 0.00 mm, vias 2 -> 0
- net VHIGH20: track 67.9 -> 0.00 mm, vias 2 -> 0
- net VHIGH22: track 67.9 -> 0.00 mm, vias 2 -> 0
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- removed copper zone on layer 1, net GND20
- removed copper zone on layer 16, net GND20
- removed copper zone on layer 1, net GND21
- removed copper zone on layer 16, net GND21
- removed copper zone on layer 1, net GND22
- removed copper zone on layer 16, net GND22
- removed copper zone on layer 1, net GND23
- removed copper zone on layer 16, net GND23
- removed copper zone on layer 1, net GND24
- removed copper zone on layer 16, net GND24
Other:
- board size 302.8 x 142.7 mm -> 142.7 x 243.8 mm
- board text added: "route out"
